Commit message: Still setting up. Playing with the stls. need to have simple test for training first. platform

File: assets/maze.urdf (robot description, URDF)
Before this commit: robot maze, 1 links, 0 joints
Links:
- link maze_link: geometry collision mesh filename=maze2.stl scale=1.5 1.5 .5; visual mesh filename=maze2.stl scale=1.5 1.5 .5
